File: pcbs/movement-control/movement-control.kicad_sch (KiCad schematic)
At the start: 1 part

Commit message: Add PCB design for control module
Parts:
- added A?: TMC2208_module, Module:Pololu_Breakout-16_15.2x20.3mm, symbol Driver_Motor:Pololu_Breakout_A4988
- added C? (x5): 100n, symbol Device:C
- added C?: 1u, symbol Device:C
- added C? (x4): 47u, symbol Device:C
- added J?: SWD PIN, symbol Connector_Generic:Conn_01x05
- added J? (x2): Conn_01x06_Male, symbol Connector:Conn_01x06_Male
- added J?: Stepper_motor_out, symbol Connector_Generic:Conn_01x04
- added J?: PWR_input, Connector:FanPinHeader_1x03_P2.54mm_Vertical, symbol Connector:Conn_01x03_Male
- added R? (x4): R, symbol Device:R
- added R?: 10k, symbol Device:R
- added R?: 100, symbol Device:R
- added R?: 100k, symbol Device:R
- added SW?: SW_RST, symbol Switch:SW_Push
- added U? (x2): BD6220F-E2, SOP8_ROM, symbol motor-driver:BD6220F-E2
Connections:
- net GND: now reaches U?.23 (VSS)
- net GND: now also U?.35 (VSS), U?.47 (VSS), U?.8 (VSSA), A?.1 (GND), A?.14 (CLK), A?.7 (GND), C?.2, C?.2, C?.2, C?.2, C?.2, C?.2, C?.2, C?.2, C?.2, C?.2, J?.3 (Pin_3), J?.5 (Pin_5), R?.1, R?.2, R?.2, R?.2, R?.2, SW?.1, U?.8 (GND), U?.8 (GND)
- net +3V3: now reaches U?.24 (VDD)
- net +3V3: now also U?.36 (VDD), U?.48 (VDD), U?.9 (VDDA), A?.10 (MS1), A?.11 (MS2), A?.2 (VDD), C?.1, C?.1, C?.1, C?.1, C?.1, C?.1, C?.1, J?.2 (Pin_2), R?.1, U?.2 (VCC), U?.2 (VCC), U?.3 (VCC), U?.3 (VCC), U?.6 (VREF), U?.6 (VREF)
- net SWDIO: now reaches U?.34 (PA13)
- net SWDIO: now also J?.1 (Pin_1)
- net SWCLK: now reaches U?.37 (PA14)
- net SWCLK: now also J?.2 (Pin_2)
- net SWO: now reaches U?.39 (PB3)
- net SWO: now also J?.3 (Pin_3)
- net BOOT0: now reaches U?.44 (BOOT0)
- net BOOT0: now also R?.2
- net NRST: now reaches U?.7 (NRST)
- net NRST: now also C?.1, J?.4 (Pin_4), R?.2
- new net: R?.1, R?.2, SW?.2
- new net +6V: A?.8 (VMOT), C?.1, C?.1, J?.1 (Pin_1)
- new net 1A: A?.4 (1A), J?.4 (Pin_4)
- new net 1B: A?.3 (1B), J?.2 (Pin_2)
- new net 2A: A?.5 (2A), J?.3 (Pin_3)
- new net 2B: A?.6 (2B), J?.1 (Pin_1)
- new net ENCODER_LEFT_A_PHASE: J?.3 (Pin_3)
- new net ENCODER_LEFT_B_PHASE: J?.4 (Pin_4)
- new net ENCODER_MINUS_RIGHT: J?.5 (Pin_5)
- new net ENCODER_PLUS_LEFT: J?.2 (Pin_2), J?.5 (Pin_5)
- new net ENCODER_PLUS_RIGHT: J?.2 (Pin_2)
- new net ENCODER_RIGHT_A_PHASE: J?.3 (Pin_3)
- new net ENCODER_RIGHT_B_PHASE: J?.4 (Pin_4)
- new net SERVO_CTRL_LEFT_FORWARD: R?.1, U?.4 (FIN)
- new net SERVO_CTRL_LEFT_OUT_1: J?.1 (Pin_1), U?.1 (OUT1)
- new net SERVO_CTRL_LEFT_OUT_2: J?.6 (Pin_6), U?.7 (OUT2)
- new net SERVO_CTRL_LEFT_REVERSE: R?.1, U?.5 (RIN)
- new net SERVO_CTRL_RIGHT_FORWARD: R?.1, U?.4 (FIN)
- new net SERVO_CTRL_RIGHT_OUT_1: J?.1 (Pin_1), U?.1 (OUT1)
- new net SERVO_CTRL_RIGHT_OUT_2: J?.6 (Pin_6), U?.7 (OUT2)
- new net SERVO_CTRL_RIGHT_REVERSE: R?.1, U?.5 (RIN)
- new net TMC_DIR: A?.16 (DIR)
- new net TMC_ENABLE: A?.9 (~{ENABLE})
- new net TMC_PDN_UART: A?.12 (PDN_UART), A?.13 (PDN_UART)
- new net TMC_STEP: A?.15 (STEP)
- no-connect marks 0 -> 35
Other:
- note added: "3x VDD capacitors + VDDA capacitor"
- note added: "BOOT"
- note added: "MANUAL RESET"
- note added: "MCU"
- note added: "MCU capacitor"
- note added: "PWR input"
- note added: "STM32 microcontroller"
- note added: "SW debug connector"
- note added: "Sepper motor capacitors"
- note added: "Servo Motor"
- note added: "Servo connectors"
- note added: "Servo control stabilizer resistors"
- note added: "Servo drive capacitors"
- note added: "Servo motor drivers"
- note added: "Steper motor out"
- note added: "Stepper motor"
- note added: "Stepper motor drive"
- note added: "VBAT cask akkor kell ha elmegy a táp, ezzel majd később foglalkozunk"
- title: (none) -> Motor Control Board
- moved on the sheet: U?

Commit message: Reposition schematic elements
Other:
- moved on the sheet: C?, J?, R?, U?

Commit message: Add capacitor to stepper motor driver, and add pdf schematic
Parts:
- added C?: 100n, symbol Device:C
Connections:
- net +3V3: now also C?.1
- net GND: now also C?.2
Changed lines of the file:
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@@
+    (pin "1")
+  )
+  (symbol (lib_id "power:+3V3") (at 276.225 21.59 0) (unit 1)
+    (in_bom yes) (on_board yes) (fields_autoplaced)
+    (property "Reference" "#PWR?" (id 0) (at 276.225 25.4 0)
+      (effects (font (size 1.27 1.27)) hide)
+    )
+    (property "Value" "+3V3" (id 1) (at 276.225 16.51 0))
+    (property "Footprint" "" (id 2) (at 276.225 21.59 0)
+      (effects (font (size 1.27 1.27)) hide)
+    )
+    (property "Datasheet" "" (id 3) (at 276.225 21.59 0)
+      (effects (font (size 1.27 1.27)) hide)
+    )
     (pin "1")
   )
@@
     (pin "2")
   )
+  (symbol (lib_id "power:GND") (at 276.225 29.21 0) (unit 1)
+    (in_bom yes) (on_board yes) (fields_autoplaced)
+    (property "Reference" "#PWR?" (id 0) (at 276.225 35.56 0)
+      (effects (font (size 1.27 1.27)) hide)
+    )
+    (property "Value" "GND" (id 1) (at 276.225 34.29 0))
+    (property "Footprint" "" (id 2) (at 276.225 29.21 0)
+      (effects (font (size 1.27 1.27)) hide)
+    )
+    (property "Datasheet" "" (id 3) (at 276.225 29.21 0)
+      (effects (font (size 1.27 1.27)) hide)
+    )
+    (pin "1")
+  )
+  (symbol (lib_id "Device:C") (at 276.225 25.4 0) (unit 1)
+    (in_bom yes) (on_board yes)
+    (property "Reference" "C?" (id 0) (at 277.495 22.86 0)
+      (effects (font (size 1.27 1.27)) (justify left))
+    )
+    (property "Value" "100n" (id 1) (at 276.225 27.94 0)
+      (effects (font (size 1.27 1.27)) (justify left))
+    )
+    (property "Footprint" "" (id 2) (at 277.1902 29.21 0)
+      (effects (font (size 1.27 1.27)) hide)
+    )
+    (property "Datasheet" "~" (id 3) (at 276.225 25.4 0)
+      (effects (font (size 1.27 1.27)) hide)
+    )
+    (pin "1")
+    (pin "2")
+  )
   (symbol (lib_id "power:+3V3") (at 43.18 161.925 0) (unit 1)
     (in_bom yes) (on_board yes) (fields_autoplaced)
@@
       (reference "#PWR?") (unit 1) (value "GND") (footprint "")
     )
+    (path "/7764b1a7-b9be-4d0c-ae2b-ec64c2b9ca7c"
+      (reference "#PWR?") (unit 1) (value "+3V3") (footprint "")
+    )
     (path "/7d3d56a8-0bd7-4b2b-b999-79d2a13d2ba0"
       (reference "#PWR?") (unit 1) (value "GND") (footprint "")
@@
     )
     (path "/ab45da5a-7864-47b0-b00b-38121fad767a"
+      (reference "#PWR?") (unit 1) (value "GND") (footprint "")
+    )
+    (path "/bde06726-cef4-4003-a1b5-ea6b7a6034a0"
       (reference "#PWR?") (unit 1) (value "GND") (footprint "")
     )
@@
       (reference "C?") (unit 1) (value "100n") (footprint "")
     )
+    (path "/c0eb397c-0f0a-48f2-a4a7-a39c38857565"
+      (reference "C?") (unit 1) (value "100n") (footprint "")
+    )

Commit message: Apend parts list, and finish schematics
Parts:
- added C?: 100n, symbol Device:C
- added D?: LED, symbol Device:LED
- added J?: SENSOR_CONNECTOR_3, symbol Connector:Conn_01x05_Male
- added J?: SENSOR_CONNECTOR_4, symbol Connector:Conn_01x05_Male
- added J?: DEBUG_UART, symbol Connector:Conn_01x04_Male
- added J?: SENSOR_CONNECTOR_2, symbol Connector:Conn_01x05_Male
- added J?: RASPBERRY_CONNECTOR, symbol Connector:Conn_01x03_Male
- added J?: SENSOR_CONNECTOR_1, symbol Connector:Conn_01x05_Male
- added R? (x4): 4.7k, symbol Device:R
- added R?: 10k, symbol Device:R
- added R?: 100k, symbol Device:R
- added R?: 1k, symbol Device:R
- added R?: 100, symbol Device:R
- added SW?: SW_RST, symbol Switch:SW_Push
- R? (x4): value R -> 10k
Connections:
- net ENCODER_MINUS_RIGHT is gone; now on net +3V3: J?.5 (Pin_5)
- net ENCODER_PLUS_LEFT is gone; now on net +3V3: J?.2 (Pin_2), J?.5 (Pin_5)
- net ENCODER_PLUS_RIGHT is gone; now on net +3V3: J?.2 (Pin_2)
- net GND is gone; now on net +3V3: A?.1 (GND), A?.14 (CLK), A?.7 (GND), C?.2, C?.2, C?.2, C?.2, C?.2, C?.2, C?.2, C?.2, C?.2, C?.2, C?.2, J?.3 (Pin_3), J?.5 (Pin_5), R?.1, R?.2, R?.2, R?.2, R?.2, SW?.1, U?.23 (VSS), U?.35 (VSS), U?.47 (VSS), U?.8 (GND), U?.8 (GND), U?.8 (VSSA)
- net +3V3: now also U?.1 (VBAT), C?.2, D?.1 (K), J?.1 (Pin_1), J?.1 (Pin_1), J?.1 (Pin_1), J?.1 (Pin_1), J?.1 (Pin_1), J?.2 (Pin_2), J?.2 (Pin_2), J?.2 (Pin_2), J?.2 (Pin_2), J?.2 (Pin_2), J?.3 (Pin_3), R?.1, R?.1, R?.1, R?.1, R?.1, R?.1, SW?.1
- net ENCODER_LEFT_A_PHASE: now also U?.10 (PA0)
- net ENCODER_LEFT_B_PHASE: now also U?.11 (PA1)
- net ENCODER_RIGHT_A_PHASE: now also U?.16 (PA6)
- net ENCODER_RIGHT_B_PHASE: now also U?.17 (PA7)
- net SERVO_CTRL_LEFT_FORWARD: now also U?.31 (PA10)
- net SERVO_CTRL_LEFT_REVERSE: now also U?.32 (PA11)
- net SERVO_CTRL_RIGHT_FORWARD: now also U?.29 (PA8)
- net SERVO_CTRL_RIGHT_REVERSE: now also U?.30 (PA9)
- net TMC_DIR: now also U?.20 (PB2)
- net TMC_PDN_UART: now also U?.42 (PB6)
- net TMC_STEP: now also U?.19 (PB1)
- net UART_TX: now reaches U?.12 (PA2)
- net UART_TX: now also J?.4 (Pin_4)
- net UART_RX: now reaches U?.13 (PA3)
- net UART_RX: now also J?.3 (Pin_3)
- net LED_0: now reaches U?.14 (PA4)
- net LED_0: now also R?.1
- net BTN_0: now reaches U?.15 (PA5)
- net BTN_0: now also C?.1, R?.2
- net I2C2_SCL: now reaches U?.21 (PB10)
- net I2C2_SCL: now also J?.2 (Pin_2), R?.2
- net I2C2_SDA: now reaches U?.22 (PB11)
- net I2C2_SDA: now also J?.1 (Pin_1), R?.2
- net SHUT_1: now reaches U?.25 (PB12)
- net SHUT_1: now also J?.5 (Pin_5)
- net SHUT_2: now reaches U?.26 (PB13)
- net SHUT_2: now also J?.5 (Pin_5)
- net SHUT_3: now reaches U?.27 (PB14)
- net SHUT_3: now also J?.5 (Pin_5)
- net SHUT_4: now reaches U?.28 (PB15)
- net SHUT_4: now also J?.5 (Pin_5)
- net I2C1_SCL: now reaches U?.45 (PB8)
- net I2C1_SCL: now also J?.4 (Pin_4), J?.4 (Pin_4), J?.4 (Pin_4), J?.4 (Pin_4), R?.2
- net I2C1_SDA: now reaches U?.46 (PB9)
- net I2C1_SDA: now also J?.3 (Pin_3), J?.3 (Pin_3), J?.3 (Pin_3), J?.3 (Pin_3), R?.2
- net TMC_ENABLE: no longer names the net of A?.9 (~{ENABLE})
- net TMC_ENABLE: now also R?.2
- new net: R?.1, R?.2, SW?.2
- new net: D?.2 (A), R?.2
- no-connect marks 35 -> 11
Other:
- note added: "Basic Peripherals"
- note added: "Encoder PWR"
- note added: "I2C BUS RASPBERRY"
- note added: "I2C BUS SENSORS"
- note added: "Raspberry Connector"
- note added: "SENSOR CONNECTORS"
- note removed: "VBAT cask akkor kell ha elmegy a táp, ezzel majd később foglalkozunk"
- moved on the sheet: A?, C?, J?, R?, SW?, U?

Commit message: Add power supply pcb layout
Parts:
- gave numbers to parts that had none: 45
