File: pcbs/movement-control/movement-control.kicad_sch (KiCad schematic)
At the start: 45 parts, among them J1 Conn_01x06_Male, J10 DEBUG_UART, J11 Stepper_motor_out, J2 Conn_01x06_Male, J3 SWD PIN, J4 SENSOR_CONNECTOR_1, J5 RASPBERRY_CONNECTOR, J6 SENSOR_CONNECTOR_2, J7 PWR_input, J8 SENSOR_CONNECTOR_3, J9 SENSOR_CONNECTOR_4, SW1 SW_RST, SW2 SW_RST, U1 BD6220F-E2, U2 BD6220F-E2, U3 STM32F103C8Tx

Commit message: Add footprints to ctrl board
Parts:
- SW2: value SW_RST -> (none)
- U1, U2: footprint SOP8_ROM -> (none)
Changed lines of the file:
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@@
       (effects (font (size 1.524 1.524)))
     )
-    (property "Footprint" "SOP8_ROM" (id 2) (at 44.45 167.005 0)
+    (property "Footprint" "" (id 2) (at 44.45 167.005 0)
       (effects (font (size 1.524 1.524)) hide)
     )
@@
       (effects (font (size 1.27 1.27)) (justify right))
     )
-    (property "Value" "SW_RST" (id 1) (at 243.967 108.204 90)
+    (property "Value" "" (id 1) (at 243.967 108.204 90)
       (effects (font (size 1.27 1.27)) (justify right))
     )
@@
       (effects (font (size 1.524 1.524)))
     )
-    (property "Footprint" "SOP8_ROM" (id 2) (at 44.45 132.715 0)
+    (property "Footprint" "" (id 2) (at 44.45 132.715 0)
       (effects (font (size 1.524 1.524)) hide)
     )
@@
     )
     (path "/108c26ac-7da2-4fb0-814e-cf4d984114ed"
-      (reference "C1") (unit 1) (value "100n") (footprint "")
+      (reference "C1") (unit 1) (value "100n") (footprint "Capacitor_SMD:C_0805_2012Metric_Pad1.18x1.45mm_HandSolder")
     )
     (path "/c8cf6ff3-a8f2-401b-a782-a36d18e3e6a7"
@@
     )
     (path "/b3ff7e4d-d66b-4d34-a49a-219b4999ec0b"
-      (reference "C3") (unit 1) (value "100n") (footprint "")
+      (reference "C3") (unit 1) (value "100n") (footprint "Capacitor_SMD:C_0805_2012Metric_Pad1.18x1.45mm_HandSolder")
     )
     (path "/ad8fe556-7ebe-46a2-88ec-7205782093b6"
-      (reference "C4") (unit 1) (value "100n") (footprint "")
+      (reference "C4") (unit 1) (value "100n") (footprint "Capacitor_SMD:C_0805_2012Metric_Pad1.18x1.45mm_HandSolder")
     )
     (path "/e5bc6e6d-d180-4499-a93e-a4c038ffdd89"
@@
     )
     (path "/42f19d25-9971-4a95-988b-64cb9dd8fdc0"
-      (reference "C6") (unit 1) (value "100n") (footprint "")
+      (reference "C6") (unit 1) (value "100n") (footprint "Capacitor_SMD:C_0805_2012Metric_Pad1.18x1.45mm_HandSolder")
     )
     (path "/265023aa-53cd-4dd4-b761-7faa486d62b0"
-      (reference "C7") (unit 1) (value "100n") (footprint "")
+      (reference "C7") (unit 1) (value "100n") (footprint "Capacitor_SMD:C_0805_2012Metric_Pad1.18x1.45mm_HandSolder")
     )
     (path "/1b0cc1c7-2221-4c1c-ad4b-ec99c2f7e327"
-      (reference "C8") (unit 1) (value "1u") (footprint "")
+      (reference "C8") (unit 1) (value "1u") (footprint "Capacitor_SMD:C_0805_2012Metric_Pad1.18x1.45mm_HandSolder")
     )
     (path "/fc0bde53-f99a-44a3-81a3-dbb81e9c5778"
-      (reference "C9") (unit 1) (value "100n") (footprint "")
+      (reference "C9") (unit 1) (value "100n") (footprint "Capacitor_SMD:C_0805_2012Metric_Pad1.18x1.45mm_HandSolder")
     )
     (path "/a57410fe-cab7-4e34-b7ad-52d6a70a6930"
@@
     )
     (path "/c0eb397c-0f0a-48f2-a4a7-a39c38857565"
-      (reference "C12") (unit 1) (value "100n") (footprint "")
+      (reference "C12") (unit 1) (value "100n") (footprint "Capacitor_SMD:C_0805_2012Metric_Pad1.18x1.45mm_HandSolder")
     )
     (path "/7c656ff7-2526-43f7-8558-c34d84ae917b"
-      (reference "D1") (unit 1) (value "LED") (footprint "")
+      (reference "D1") (unit 1) (value "LED") (footprint "LED_SMD:LED_0805_2012Metric_Pad1.15x1.40mm_HandSolder")
     )
     (path "/1cd616c3-06dd-4d25-9068-781ff43961db"
@@
     )
     (path "/fd249575-fefc-401e-8259-147497dc7ccb"
-      (reference "SW1") (unit 1) (value "SW_RST") (footprint "")
+      (reference "SW1") (unit 1) (value "SW_RST") (footprint "Button_Switch_SMD:SW_Push_1P1T_NO_6x6mm_H9.5mm")
     )
     (path "/ab2a858a-f5aa-475b-b833-babe4a38f3ae"
-      (reference "SW2") (unit 1) (value "SW_RST") (footprint "")
+      (reference "SW2") (unit 1) (value "SW_BTN") (footprint "Button_Switch_SMD:SW_Push_1P1T_NO_6x6mm_H9.5mm")
     )
     (path "/cfa0cc3f-16c9-47dc-8f68-6b658d60fd31"
-      (reference "U1") (unit 1) (value "BD6220F-E2") (footprint "SOP8_ROM")
+      (reference "U1") (unit 1) (value "BD6220F-E2") (footprint "Package_SO:SOP-8_3.9x4.9mm_P1.27mm")
     )
     (path "/28e55824-6f25-4325-ad7c-a821934d9e90"
-      (reference "U2") (unit 1) (value "BD6220F-E2") (footprint "SOP8_ROM")
+      (reference "U2") (unit 1) (value "BD6220F-E2") (footprint "Package_SO:SOP-8_3.9x4.9mm_P1.27mm")
     )
     (path "/adcbf4d0-ed9c-4c7d-b78f-3bcbe974bdcb"

Commit message: Add auto saved files to gitignore
Fix motor driver power inputs.
Add PWR_FLAGs to 3V3, 6V and GND
Parts:
- C1, C12, C3, C4, C6, C7, C8, C9: footprint (none) -> Capacitor_SMD:C_0805_2012Metric_Pad1.18x1.45mm_HandSolder
- D1: footprint (none) -> LED_SMD:LED_0805_2012Metric_Pad1.15x1.40mm_HandSolder
- R1, R10, R11, R12, R13, R14, R15, R2, R3, R4, R5, R6, R7, R8, R9: footprint (none) -> Resistor_SMD:R_0805_2012Metric_Pad1.20x1.40mm_HandSolder
- SW1: footprint (none) -> Button_Switch_SMD:SW_Push_1P1T_NO_6x6mm_H9.5mm
- SW2: value (none) -> SW_BTN; footprint (none) -> Button_Switch_SMD:SW_Push_1P1T_NO_6x6mm_H9.5mm
- U1, U2: footprint (none) -> Package_SO:SOP-8_3.9x4.9mm_P1.27mm
Connections:
- net +3V3: no longer U1.2 (VCC), U1.3 (VCC), U2.2 (VCC), U2.3 (VCC)
- net +6V: now also U1.2 (VCC), U1.3 (VCC), U2.2 (VCC), U2.3 (VCC)
Other:
- note added: "PWR flags"
- moved on the sheet: U2

Commit message: Fix servo driver capacitors
connected to 3v3 instead of 6V
Connections:
- net +3V3: no longer C2.1, C5.1
- net +6V: now also C2.1, C5.1
Other:
- moved on the sheet: C2, C5

Commit message: Fix wrong name for servo motor connectors
Parts:
- J1, J2: value Conn_01x06_Male -> (none)
Changed lines of the file:
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@@
       (effects (font (size 1.27 1.27)) (justify right))
     )
-    (property "Value" "Conn_01x06_Male" (id 1) (at 148.59 163.195 0)
+    (property "Value" "" (id 1) (at 151.13 163.83 0)
       (effects (font (size 1.27 1.27)) (justify right))
     )
@@
       (effects (font (size 1.27 1.27)) (justify right))
     )
-    (property "Value" "Conn_01x06_Male" (id 1) (at 148.59 182.88 0)
+    (property "Value" "" (id 1) (at 149.86 182.88 0)
       (effects (font (size 1.27 1.27)) (justify right))
     )
@@
   (symbol (lib_id "power:+6V") (at 135.89 128.27 0) (unit 1)
     (in_bom yes) (on_board yes) (fields_autoplaced)
-    (property "Reference" "#PWR?" (id 0) (at 135.89 132.08 0)
+    (property "Reference" "#PWR0156" (id 0) (at 135.89 132.08 0)
       (effects (font (size 1.27 1.27)) hide)
     )
@@
   (symbol (lib_id "power:+6V") (at 144.78 128.27 0) (unit 1)
     (in_bom yes) (on_board yes) (fields_autoplaced)
-    (property "Reference" "#PWR?" (id 0) (at 144.78 132.08 0)
+    (property "Reference" "#PWR0160" (id 0) (at 144.78 132.08 0)
       (effects (font (size 1.27 1.27)) hide)
     )
@@
       (reference "#PWR0155") (unit 1) (value "GND") (footprint "")
     )
+    (path "/9ccbfdf6-7fca-4850-a349-a9950c8e630e"
+      (reference "#PWR0156") (unit 1) (value "+6V") (footprint "")
+    )
     (path "/deb8cb37-e974-4b2b-950f-469f47de51e6"
       (reference "#PWR0157") (unit 1) (value "GND") (footprint "")
@@
       (reference "#PWR0159") (unit 1) (value "GND") (footprint "")
     )
+    (path "/fad950b4-5ebf-4143-95cd-a0ab1ac5bc4c"
+      (reference "#PWR0160") (unit 1) (value "+6V") (footprint "")
+    )
     (path "/d78a485f-9cc1-4769-b49d-4b1c97dee49a"
       (reference "#PWR0161") (unit 1) (value "+3V3") (footprint "")
@@
       (reference "#PWR0169") (unit 1) (value "+6V") (footprint "")
     )
-    (path "/9ccbfdf6-7fca-4850-a349-a9950c8e630e"
-      (reference "#PWR?") (unit 1) (value "+6V") (footprint "")
-    )
-    (path "/fad950b4-5ebf-4143-95cd-a0ab1ac5bc4c"
-      (reference "#PWR?") (unit 1) (value "+6V") (footprint "")
-    )
     (path "/7dbb1359-f267-4d5a-b7ae-25f0e3894c63"
       (reference "A1") (unit 1) (value "TMC2208_module") (footprint "Module:Pololu_Breakout-16_15.2x20.3mm")
@@
     )
     (path "/1cd616c3-06dd-4d25-9068-781ff43961db"
-      (reference "J1") (unit 1) (value "Conn_01x06_Male") (footprint "")
+      (reference "J1") (unit 1) (value "CONN_SERVO_RIGHT") (footprint "")
     )
     (path "/5da34ef7-ba7c-4e70-a24c-f1b432b4b931"
-      (reference "J2") (unit 1) (value "Conn_01x06_Male") (footprint "")
+      (reference "J2") (unit 1) (value "CONN_SERVO_LEFT") (footprint "")
     )
     (path "/16c09044-1165-4770-b343-a0df4cb8ff11"

Commit message: Modify SWD connector schematic, and add correct footprints
Parts:
- removed J3: SWD PIN, symbol Connector_Generic:Conn_01x05
- added J12: SWD_CONNECTOR, Connector_PinHeader_2.54mm:PinHeader_2x05_P2.54mm_Vertical, symbol Connector_Generic:Conn_02x05_Odd_Even
- C10, C11, C2, C5: footprint (none) -> Capacitor_SMD:C_0805_2012Metric_Pad1.18x1.45mm_HandSolder
- J1: value (none) -> CONN_SERVO_RIGHT; footprint (none) -> Connector_PinHeader_2.54mm:PinHeader_1x06_P2.54mm_Horizontal
- J10: footprint (none) -> Connector_PinHeader_2.54mm:PinHeader_1x04_P2.54mm_Vertical
- J11: footprint (none) -> Connector_PinHeader_2.54mm:PinHeader_1x04_P2.54mm_Horizontal
- J2: value (none) -> CONN_SERVO_LEFT; footprint (none) -> Connector_PinHeader_2.54mm:PinHeader_1x06_P2.54mm_Horizontal
- J4, J6, J8, J9: footprint (none) -> Connector_PinHeader_2.54mm:PinHeader_1x05_P2.54mm_Horizontal
- J5: footprint (none) -> Connector_PinHeader_2.54mm:PinHeader_1x03_P2.54mm_Horizontal
- J7: footprint Connector:FanPinHeader_1x03_P2.54mm_Vertical -> Connector_PinHeader_2.54mm:PinHeader_1x03_P2.54mm_Horizontal
Connections:
- net +3V3: now also J12.10 (Pin_10), J12.2 (Pin_2), J12.4 (Pin_4), J12.6 (Pin_6), J12.8 (Pin_8)
- net NRST: now also J12.9 (Pin_9)
- net SWCLK: now also J12.3 (Pin_3)
- net SWDIO: now also J12.1 (Pin_1)
- net SWO: now also J12.7 (Pin_7)
- no-connect marks 11 -> 12
Other:
- moved on the sheet: C1, C3, C6, C7, U1, U2

Commit message: Fix connected power and gnd
Connected power and gnd fixed in motor output power labels. Also PWR flags were removed, and power outputs were created at PWR_CONNECTOR
Parts:
- U2: value BD6220F-E2 -> (none); footprint Package_SO:SOP-8_3.9x4.9mm_P1.27mm -> (none)
- U3: value STM32F103C8Tx -> (none); footprint Package_QFP:LQFP-48_7x7mm_P0.5mm -> (none)
Connections:
- net +3V3: no longer A1.1 (GND), A1.14 (CLK), A1.7 (GND), C1.2, C10.2, C11.2, C12.2, C2.2, C3.2, C4.2, C5.2, C6.2, C7.2, C8.2, C9.2, D1.1 (K), J1.5 (Pin_5), J10.2 (Pin_2), J12.10 (Pin_10), J12.2 (Pin_2), J12.4 (Pin_4), J12.6 (Pin_6), J12.8 (Pin_8), J4.2 (Pin_2), J5.3 (Pin_3), J6.2 (Pin_2), J7.3 (Pin_3), J8.2 (Pin_2), J9.2 (Pin_2), R1.2, R2.2, R3.2, R4.2, R7.1, R8.1, SW1.1, SW2.1, U1.8 (GND), U2.8 (GND), U3.23 (VSS), U3.35 (VSS), U3.47 (VSS), U3.8 (VSSA)
- new net GND: A1.1 (GND), A1.14 (CLK), A1.7 (GND), C1.2, C10.2, C11.2, C12.2, C2.2, C3.2, C4.2, C5.2, C6.2, C7.2, C8.2, C9.2, D1.1 (K), J1.5 (Pin_5), J10.2 (Pin_2), J12.10 (Pin_10), J12.2 (Pin_2), J12.4 (Pin_4), J12.6 (Pin_6), J12.8 (Pin_8), J4.2 (Pin_2), J5.3 (Pin_3), J6.2 (Pin_2), J7.3 (Pin_3), J8.2 (Pin_2), J9.2 (Pin_2), R1.2, R2.2, R3.2, R4.2, R7.1, R8.1, SW1.1, SW2.1, U1.8 (GND), U2.8 (GND), U3.23 (VSS), U3.35 (VSS), U3.47 (VSS), U3.8 (VSSA)
Other:
- note removed: "PWR flags"
- moved on the sheet: J5

Commit message: Fix motor signal bug, and add footprint to movement-control
Parts:
- U2: value (none) -> BD6220F-E2; footprint (none) -> Package_SO:SOP-8_3.9x4.9mm_P1.27mm
- U3: value (none) -> STM32F103C8Tx; footprint (none) -> Package_QFP:LQFP-48_7x7mm_P0.5mm
Connections:
- net +3V3: no longer J2.5 (Pin_5)
- net GND: now also J2.5 (Pin_5)
Changed lines of the file:
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@@
     (effects (font (size 1.27 1.27)) (justify left bottom))
   )
-  (label "ENCODER_PLUS_LEFT" (at 141.605 178.435 0)
+  (label "ENCODER_MINUS_LEFT" (at 141.605 178.435 0)
     (effects (font (size 1.27 1.27)) (justify left bottom))
   )
@@
       (effects (font (size 1.524 1.524)))
     )
-    (property "Value" "" (id 1) (at 64.77 188.595 0)
+    (property "Value" "BD6220F-E2" (id 1) (at 64.77 188.595 0)
       (effects (font (size 1.524 1.524)))
     )
-    (property "Footprint" "" (id 2) (at 44.45 168.275 0)
+    (property "Footprint" "Package_SO:SOP-8_3.9x4.9mm_P1.27mm" (id 2) (at 44.45 168.275 0)
       (effects (font (size 1.524 1.524)) hide)
     )
@@
       (effects (font (size 1.27 1.27)) (justify left))
     )
-    (property "Value" "" (id 1) (at 54.61 102.362 0)
-      (effects (font (size 1.27 1.27)) (justify left))
-    )
-    (property "Footprint" "" (id 2) (at 35.56 100.584 0)
+    (property "Value" "STM32F103C8Tx" (id 1) (at 54.61 102.362 0)
+      (effects (font (size 1.27 1.27)) (justify left))
+    )
+    (property "Footprint" "Package_QFP:LQFP-48_7x7mm_P0.5mm" (id 2) (at 35.56 100.584 0)
       (effects (font (size 1.27 1.27)) (justify right) hide)
     )
