File: pcbs/power-supply-unit/power-supply-unit.kicad_sch (KiCad schematic)
At the start: 18 parts

Commit message: Add connectors and organize PWR supply schematic
Parts:
- added J?: PWR_CONN_RASPI, symbol Connector:Conn_01x02_Male
- added J?: PWR_CONN_CTRL, symbol Connector:Conn_01x03_Male
Connections:
- net +3V3: now also J?.2 (Pin_2)
- net +5V: now also J?.1 (Pin_1)
- net +6V: now also J?.1 (Pin_1)
- net GND: now also J?.2 (Pin_2), J?.3 (Pin_3)
Other:
- note added: "12V"
- note added: "BMS"
- note added: "BMS output"
- note added: "Buck converter 5V"
- note added: "Buck converter 6V"
- note added: "GND"
- note added: "PWR connector to control module"
- note added: "PWR connector to raspberry pi"
- note added: "Regulated 3V3 supply"
- moved on the sheet: C?, D?, J?, L?, R?, U?

Commit message: Update gitignore
Parts:
- C1, C2, C5, C6: renamed from C?; footprint (none) -> Capacitor_SMD:C_0805_2012Metric_Pad1.18x1.45mm_HandSolder
- C3, C4: renamed from C?; footprint (none) -> Capacitor_SMD:C_Elec_6.3x7.7
- D1, D2: renamed from D?; footprint (none) -> Diode_THT:D_DO-201AD_P15.24mm_Horizontal
- J1, J2: renamed from J?; footprint (none) -> Connector_PinHeader_2.54mm:PinHeader_1x02_P2.54mm_Horizontal
- J3: renamed from J?; footprint (none) -> Connector_PinHeader_2.54mm:PinHeader_1x03_P2.54mm_Horizontal
- L1, L2: renamed from L?; footprint (none) -> Inductor_SMD:L_Fastron_PISR_Handsoldering
- R1, R2, R3, R4: renamed from R?; footprint (none) -> Resistor_SMD:R_0805_2012Metric_Pad1.20x1.40mm_HandSolder
- gave numbers to parts that had none: 3

Commit message: Redesign PWR supply to match real part footprints
Parts:
- C1, C2: footprint Capacitor_SMD:C_0805_2012Metric_Pad1.18x1.45mm_HandSolder -> Capacitor_SMD:C_Elec_6.3x7.7
- C3, C4: footprint Capacitor_SMD:C_Elec_6.3x7.7 -> Capacitor_SMD:C_Elec_10x10.2
Changed lines of the file:
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@@
       (effects (font (size 1.27 1.27)) (justify left))
     )
-    (property "Footprint" "Capacitor_SMD:C_Elec_6.3x7.7" (id 2) (at 95.4532 109.22 0)
+    (property "Footprint" "Capacitor_SMD:C_Elec_10x10.2" (id 2) (at 95.4532 109.22 0)
       (effects (font (size 1.27 1.27)) hide)
     )
@@
       (effects (font (size 1.27 1.27)) (justify left))
     )
-    (property "Footprint" "Capacitor_SMD:C_0805_2012Metric_Pad1.18x1.45mm_HandSolder" (id 2) (at 42.3672 72.898 0)
+    (property "Footprint" "Capacitor_SMD:C_Elec_6.3x7.7" (id 2) (at 42.3672 72.898 0)
       (effects (font (size 1.27 1.27)) hide)
     )
@@
       (effects (font (size 1.27 1.27)) (justify left))
     )
-    (property "Footprint" "Capacitor_SMD:C_Elec_6.3x7.7" (id 2) (at 95.4532 73.914 0)
+    (property "Footprint" "Capacitor_SMD:C_Elec_10x10.2" (id 2) (at 95.4532 73.914 0)
       (effects (font (size 1.27 1.27)) hide)
     )
@@
       (effects (font (size 1.27 1.27)) (justify left))
     )
-    (property "Footprint" "Capacitor_SMD:C_0805_2012Metric_Pad1.18x1.45mm_HandSolder" (id 2) (at 42.3672 108.204 0)
+    (property "Footprint" "Capacitor_SMD:C_Elec_6.3x7.7" (id 2) (at 42.3672 108.204 0)
       (effects (font (size 1.27 1.27)) hide)
     )
@@
     )
     (path "/8ab3c70e-be6e-4202-8f32-8f153784e0d8"
-      (reference "C1") (unit 1) (value "100u") (footprint "Capacitor_SMD:C_0805_2012Metric_Pad1.18x1.45mm_HandSolder")
+      (reference "C1") (unit 1) (value "100u") (footprint "Capacitor_SMD:C_Elec_6.3x7.7")
     )
     (path "/c9060e2b-e22b-4871-af48-c1d48fb458a7"
-      (reference "C2") (unit 1) (value "100u") (footprint "Capacitor_SMD:C_0805_2012Metric_Pad1.18x1.45mm_HandSolder")
+      (reference "C2") (unit 1) (value "100u") (footprint "Capacitor_SMD:C_Elec_6.3x7.7")
     )
     (path "/bb641977-aea1-4a8b-8576-e6305f06a754"
-      (reference "C3") (unit 1) (value "1000u") (footprint "Capacitor_SMD:C_Elec_6.3x7.7")
+      (reference "C3") (unit 1) (value "1000u") (footprint "Capacitor_SMD:C_Elec_10x10.2")
     )
     (path "/27f87310-5247-4a35-a060-319434d04ce4"
-      (reference "C4") (unit 1) (value "1000u") (footprint "Capacitor_SMD:C_Elec_6.3x7.7")
+      (reference "C4") (unit 1) (value "1000u") (footprint "Capacitor_SMD:C_Elec_10x10.2")
     )
     (path "/2c6e9b54-fd3f-484a-b847-a46d6178c2bd"
