File: pcbs/power-supply-unit/power-supply-unit.kicad_pcb (KiCad board)
At the start: 2 copper layers, 44.5 x 74.9 mm, 20 parts, among them J1 BMS_OUTPUT, J2 PWR_CONN_RASPI, J3 PWR_CONN_CTRL, U1 LM2576S-ADJ, U2 LM2576S-ADJ, U3 AMS1117-3.3

Commit message: Add power supply pcb layout
Parts:
- moved J3 16.6 mm to (142.9, 66.8)
- moved J1 9.02 mm to (113.8, 77.5)
- moved C6 2.07 mm to (134.4, 77.0)
- moved C5 1.78 mm to (133.3, 80.5)
- moved U3 1.78 mm to (139.7, 78.0)
- moved C3 1.27 mm to (133.3, 48.3)
- moved C2 1.27 mm to (113.7, 88.3)
- moved L1 1.27 mm to (133.3, 61.0)
- moved C1 0.68 mm to (113.7, 51.4)
- moved D1 0.64 mm to (117.5, 54.6)
- moved D2 0.64 mm to (117.5, 91.4)
- moved R1 0.64 mm to (126.4, 53.3)
- moved R3 0.64 mm to (126.4, 90.2)
- moved R2 0.63 mm to (122.6, 53.3)
- moved R4 0.63 mm to (122.6, 90.2)
Routing:
- net +5V: track 0.00 -> 23.2 mm
- net +3V3: track 0.00 -> 18.3 mm
- net GND: track 0.00 -> 9.91 mm, vias 0 -> 246
- net Net-(R3-Pad2): track 0.00 -> 5.70 mm
- net Net-(R1-Pad2): track 0.00 -> 5.69 mm
- added copper zone on F.Cu, net +12V
- added copper zone on F.Cu, net +5V
- added copper zone on F.Cu, net +6V
- added copper zone on B.Cu, net GND
- added copper zone on F.Cu, net GND
- added copper zone on F.Cu, net Net-(D1-Pad1)
- added copper zone on F.Cu, net Net-(D2-Pad1)
Other:
- board size 44.5 x 74.9 mm -> 34.3 x 74.9 mm

Commit message: Add mounting holes to PSU
Parts:
- added REF01: MountingHole_2.5mm, MountingHole:MountingHole_2.5mm, F.Cu at (139.7, 113.0)
- added REF02: MountingHole_2.5mm, MountingHole:MountingHole_2.5mm, F.Cu at (116.8, 113.0)
- added REF03: MountingHole_2.5mm, MountingHole:MountingHole_2.5mm, F.Cu at (141.0, 39.4)
Other:
- board size 34.3 x 74.9 mm -> 34.3 x 83.2 mm
Changed lines of the file:
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@@
     )
+  )
+  (footprint "MountingHole:MountingHole_2.5mm" (layer "F.Cu")
+    (at 140.97 39.37)
+    (descr "Mounting Hole 2.5mm, no annular")
+    (tags "mounting hole 2.5mm no annular")
+    (attr exclude_from_pos_files exclude_from_bom)
+    (fp_text reference "REF03" (at 0 -3.499993) (layer "F.SilkS") hide
+      (effects (font (size 1 1) (thickness 0.15)))
+    )
+    (fp_text value "MountingHole_2.5mm" (at 0 3.5) (layer "F.Fab")
+      (effects (font (size 1 1) (thickness 0.15)))
+    )
+    (fp_text user "${REFERENCE}" (at 0 0) (layer "F.Fab")
+      (effects (font (size 1 1) (thickness 0.15)))
+    )
+    (fp_circle (center 0 0) (end 2.5 0) (layer "Cmts.User") (width 0.15) (fill none))
+    (fp_circle (center 0 0) (end 2.75 0) (layer "F.CrtYd") (width 0.05) (fill none))
+    (pad "" np_thru_hole circle (at 0 0) (size 2.5 2.5) (drill 2.5) (layers *.Cu *.Mask))
   )
   (footprint "Capacitor_SMD:C_0805_2012Metric_Pad1.18x1.45mm_HandSolder" (layer "F.Cu")
@@
       (rotate (xyz 0 0 0))
     )
+  )
+  (footprint "MountingHole:MountingHole_2.5mm" (layer "F.Cu")
+    (at 139.7 113.03)
+    (descr "Mounting Hole 2.5mm, no annular")
+    (tags "mounting hole 2.5mm no annular")
+    (attr exclude_from_pos_files exclude_from_bom)
+    (fp_text reference "REF01" (at 0 -3.499993) (layer "F.SilkS") hide
+      (effects (font (size 1 1) (thickness 0.15)))
+    )
+    (fp_text value "MountingHole_2.5mm" (at 0 3.5) (layer "F.Fab")
+      (effects (font (size 1 1) (thickness 0.15)))
+    )
+    (fp_text user "${REFERENCE}" (at 0 0) (layer "F.Fab")
+      (effects (font (size 1 1) (thickness 0.15)))
+    )
+    (fp_circle (center 0 0) (end 2.5 0) (layer "Cmts.User") (width 0.15) (fill none))
+    (fp_circle (center 0 0) (end 2.75 0) (layer "F.CrtYd") (width 0.05) (fill none))
+    (pad "" np_thru_hole circle (at 0 0) (size 2.5 2.5) (drill 2.5) (layers *.Cu *.Mask))
+  )
+  (footprint "MountingHole:MountingHole_2.5mm" (layer "F.Cu")
+    (at 116.84 113.03)
+    (descr "Mounting Hole 2.5mm, no annular")
+    (tags "mounting hole 2.5mm no annular")
+    (attr exclude_from_pos_files exclude_from_bom)
+    (fp_text reference "REF02" (at 0 -3.499993) (layer "F.SilkS") hide
+      (effects (font (size 1 1) (thickness 0.15)))
+    )
+    (fp_text value "MountingHole_2.5mm" (at 0 3.5) (layer "F.Fab")
+      (effects (font (size 1 1) (thickness 0.15)))
+    )
+    (fp_text user "${REFERENCE}" (at 0 0) (layer "F.Fab")
+      (effects (font (size 1 1) (thickness 0.15)))
+    )
+    (fp_circle (center 0 0) (end 2.5 0) (layer "Cmts.User") (width 0.15) (fill none))
+    (fp_circle (center 0 0) (end 2.75 0) (layer "F.CrtYd") (width 0.05) (fill none))
+    (pad "" np_thru_hole circle (at 0 0) (size 2.5 2.5) (drill 2.5) (layers *.Cu *.Mask))
   )
   (footprint "Inductor_SMD:L_Fastron_PISR_Handsoldering" (layer "F.Cu")
@@
   )
   (gr_line (start 145.415 34.925) (end 111.125 34.925) (layer "Edge.Cuts") (width 0.1))
-  (gr_line (start 111.125 34.925) (end 111.125 109.855) (layer "Edge.Cuts") (width 0.1))
-  (gr_line (start 145.415 109.855) (end 145.415 34.925) (layer "Edge.Cuts") (width 0.1))
-  (gr_line (start 111.125 109.855) (end 145.415 109.855) (layer "Edge.Cuts") (width 0.1))
+  (gr_line (start 111.125 34.925) (end 111.125 118.11) (layer "Edge.Cuts") (width 0.1))
+  (gr_line (start 145.415 118.11) (end 145.415 34.925) (layer "Edge.Cuts") (width 0.1))
+  (gr_line (start 111.125 118.11) (end 145.415 118.11) (layer "Edge.Cuts") (width 0.1))
   (segment (start 134.366 75.9245) (end 136.3035 75.9245) (width 0.762) (layer "F.Cu") (net 2))
   (segment (start 121.52 86.42) (end 121.52 90.135) (width 0.762) (layer "F.Cu") (net 2))
@@
     (polygon
       (pts
-        (xy 145.542 109.982)
-        (xy 110.998 109.982)
+        (xy 145.542 118.872)
+        (xy 110.998 118.872)
         (xy 110.998 34.798)
         (xy 145.542 34.798)
@@
     (polygon
       (pts
-        (xy 145.415 109.855)
-        (xy 111.125 109.855)
+        (xy 145.415 118.745)
+        (xy 111.125 118.745)
         (xy 111.125 34.925)
         (xy 145.415 34.925)

Commit message: Redesign PWR supply to match real part footprints
Parts:
- added REF03: MountingHole_2.5mm, MountingHole:MountingHole_2.5mm, F.Cu at (110.2, 39.0)
- C1, C2: footprint Capacitor_SMD:C_0805_2012Metric_Pad1.18x1.45mm_HandSolder -> Capacitor_SMD:C_Elec_6.3x7.7
- C3, C4: footprint Capacitor_SMD:C_Elec_6.3x7.7 -> Capacitor_SMD:C_Elec_10x10.2
- moved L1 9.73 mm to (124.5, 65.0)
- moved L2 9.07 mm to (124.5, 101.0)
- moved D1 7.73 mm to (110.2, 57.4)
- moved D2 7.62 mm to (110.2, 93.9)
- moved J2 7.44 mm to (137.6, 94.7)
- moved REF02 6.88 mm to (110.2, 115.0)
- moved J3 6.87 mm to (137.6, 62.5)
- moved C6 5.28 mm to (130.0, 74.0)
- moved J1 5.01 mm to (110.0, 80.7)
- moved U3 4.75 mm to (136.0, 75.0)
- moved C5 4.19 mm to (130.0, 78.0), turned to -90 degrees
- moved REF03 3.49 mm to (137.5, 39.0)
- moved C2 3.02 mm to (110.6, 88.2)
- moved REF01 2.95 mm to (137.5, 115.0)
- moved C1 2.93 mm to (110.8, 51.8)
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Routing:
- net +5V: track 23.2 -> 2.99 mm
- net +3V3: track 18.3 -> 19.8 mm
- net GND: track 9.91 -> 10.4 mm, vias 246 -> 238
Other:
- board size 34.3 x 83.2 mm -> 37.5 x 86 mm
- board text added: "12V"
- board text added: "3V3"
- board text added: "5V"
- board text added: "6V"
- board text added: "GND"

Commit message: Fix small errors, add more stitching vias
Routing:
- net GND: vias 238 -> 313

Commit message: Minor redesign of vias on pwr supply
Routing:
- net GND: vias 313 -> 379
Other:
- board text added: "L2"

Commit message: Fix mounting hole position inaccuracy with pwr-supply
Parts:
- moved REF02 0.25 mm to (110.0, 115.0)
- moved REF03 0.25 mm to (110.0, 39.0)
